Commit message: add RT source

File: urdf/rb20_1900es.urdf (robot description, URDF)
Before this commit: robot rb20_1900es, 8 links, 7 joints
Links:
- added link link_end, mass 33.803183177691814; collision mesh filename=meshes/link_rt.stl scale=0.001 0.001 0.001; visual mesh filename=meshes/link_rt.stl scale=0.001 0.001 0.001
Joints:
- added joint joint_end: type fixed, parent link6, child link_end, origin xyz=0.0 0.0 0.13 rpy=-1.57 0 0
