Commit message: add base rail

File: urdf/rb10_1300e_DDA.urdf (robot description, URDF)
Before this commit: robot dda_rb10_1300e, 9 links, 8 joints
Links:
- added link dda_link_base_x, mass 100.0; collision box size=8.5 0.4 0.2; visual box size=8.5 0.4 0.2
Joints:
- added joint dda_joint_base_x: type prismatic, parent dda_link_base_x, child dda_link0, origin xyz=0 0 0.2 rpy=0 0 0, axis 1 0 0, limit lower=0.0 upper=8.5 effort=1000.0 velocity=1.0
- joint dda_joint_base: origin xyz=0 0 0 rpy=0 0 0 -> xyz=0 0 0 rpy=0 0 1.57079632679
