Commit message: add position colum in URDF

File: urdf/positioner.urdf (robot description, URDF)
Before this commit: robot positioner, 1 links, 0 joints
Links:
- added link column_x; collision mesh filename=meshes/positioner/collision/column_x.stl scale=0.001 0.001 0.001; visual mesh filename=meshes/positioner/visual/column_x.dae
Joints:
- added joint base_to_column_x: type prismatic, parent base_link, child column_x, origin xyz=7.907 1.377 0.328 rpy=0 0 0, axis 1 0 0, limit lower=0.0 upper=8.5 effort=1000.0 velocity=1.0

Commit message: modified urdf

File: urdf/positioner.urdf (robot description, URDF)
Before this commit: robot positioner, 2 links, 1 joints
Links:
- removed link column_x
- added link f_column_z; collision mesh filename=meshes/positioner/collision/f_column_z.stl scale=0.001 0.001 0.001; visual mesh filename=meshes/positioner/visual/f_column_z.dae
- added link m_column; collision mesh filename=meshes/positioner/collision/m_column.stl scale=0.001 0.001 0.001; visual mesh filename=meshes/positioner/visual/m_column.dae
- added link m_column_passive_r; collision mesh filename=meshes/positioner/collision/m_column_passive_r.stl scale=0.001 0.001 0.001; visual mesh filename=meshes/positioner/visual/m_column_passive_r.dae
- added link m_column_z; collision mesh filename=meshes/positioner/collision/m_column_z.stl scale=0.001 0.001 0.001; visual mesh filename=meshes/positioner/visual/m_column_z.dae
Joints:
- removed joint base_to_column_x
- added joint base_to_f_column_z: type prismatic, parent base_link, child f_column_z, origin xyz=0 0 0 rpy=0 0 0, axis 0 0 1, limit lower=0.0 upper=3.0 effort=1000.0 velocity=1.0
- added joint base_to_m_column: type prismatic, parent base_link, child m_column, origin xyz=7.907 1.377 0.328 rpy=0 0 0, axis 1 0 0, limit lower=0.0 upper=8.5 effort=1000.0 velocity=1.0
- added joint m_column_to_m_column_z: type prismatic, parent m_column, child m_column_z, origin xyz=0 0 0 rpy=0 0 0, axis 0 0 1, limit lower=0.0 upper=3.0 effort=1000.0 velocity=1.0
- added joint m_column_z_to_m_column_passive_r: type revolute, parent m_column_z, child m_column_passive_r, origin xyz=0 0 0 rpy=0 0 0, axis 0 0 1, limit lower=-3.14159 upper=3.14159 effort=1000.0 velocity=1.0

Commit message: update URDF files

File: urdf/positioner.urdf (robot description, URDF)
Before this commit: robot positioner, 5 links, 4 joints
Links:
- added link f_column_passive_clamp; collision mesh filename=meshes/positioner/collision/f_column_passive_clamp.stl scale=0.001 0.001 0.001; visual mesh filename=meshes/positioner/visual/f_column_passive_clamp.dae
- added link f_column_r; collision mesh filename=meshes/positioner/collision/f_column_r.stl scale=0.001 0.001 0.001; visual mesh filename=meshes/positioner/visual/f_column_r.dae
Joints:
- added joint f_column_r_to_f_column_passive_clamp: type prismatic, parent f_column_r, child f_column_passive_clamp, origin xyz=0.427 0.9 0.0 rpy=0 0 0, axis 0 1 0, limit lower=-0.9 upper=0.0 effort=1000.0 velocity=1.0
- added joint f_column_z_to_f_column_r: type revolute, parent f_column_z, child f_column_r, origin xyz=0.48 1.37 1.3 rpy=0 0 0, axis 1 0 0, limit lower=-3.14159 upper=3.14159 effort=1000.0 velocity=1.0
- joint base_to_f_column_z: limit lower=0.0 upper=3.0 effort=1000.0 velocity=1.0 -> lower=0.0 upper=0.85 effort=1000.0 velocity=1.0
- joint base_to_m_column: limit lower=0.0 upper=8.5 effort=1000.0 velocity=1.0 -> lower=-4.7 upper=0.0 effort=1000.0 velocity=1.0; origin xyz=7.907 1.377 0.328 rpy=0 0 0 -> xyz=8.0 1.377 0.328 rpy=0 0 0
- joint m_column_to_m_column_z: limit lower=0.0 upper=3.0 effort=1000.0 velocity=1.0 -> lower=0.0 upper=0.85 effort=1000.0 velocity=1.0; mimic (none) -> joint=base_to_f_column_z multiplier=1.0 offset=0.0
- joint m_column_z_to_m_column_passive_r: axis 0 0 1 -> 1 0 0; origin xyz=0 0 0 rpy=0 0 0 -> xyz=-0.247 0 0.885 rpy=0 0 0

File: urdf/rb10_1300e_DDA.urdf (robot description, URDF)
Before this commit: robot dda_rb10_1300e, 10 links, 9 joints
Links:
- removed link dda_link_base_x
- added link dda_link_carriage, mass 50.0; collision box size=0.4 0.5 0.1; visual box size=0.4 0.7 0.2
- added link dda_link_linear_track, mass 100.0; collision box size=8.3 0.4 0.2; visual box size=8.3 0.4 0.2
Joints:
- removed joint dda_joint_base_x
- added joint dda_joint_carriage: type prismatic, parent dda_link_carriage, child dda_link0, origin xyz=0.2 0 0.2 rpy=0 0 0, axis 0 1 0, limit lower=0.0 upper=0.5 effort=1000.0 velocity=1.0
- added joint dda_joint_linear_track: type prismatic, parent dda_link_linear_track, child dda_link_carriage, origin xyz=0 0 0.2 rpy=0 0 0, axis 1 0 0, limit lower=0.0 upper=7.9 effort=1000.0 velocity=1.0

File: urdf/rb20_1900es_RT.urdf (robot description, URDF)
Before this commit: robot rb20_1900es, 10 links, 9 joints
Links:
- removed link rt_link_base_x
- added link rt_link_carriage, mass 50.0; collision box size=0.4 0.5 0.1; visual box size=0.4 0.7 0.2
- added link rt_link_linear_track, mass 100.0; collision box size=8.3 0.4 0.2; visual box size=8.3 0.4 0.2
Joints:
- removed joint rt_joint_base_x
- added joint rt_joint_carriage: type prismatic, parent rt_link_carriage, child rt_link0, origin xyz=0.2 0 0.2 rpy=0 0 0, axis 0 1 0, limit lower=0.0 upper=0.5 effort=1000.0 velocity=1.0
- added joint rt_joint_linear_track: type prismatic, parent rt_link_linear_track, child rt_link_carriage, origin xyz=0 0 0.2 rpy=0 0 0, axis 1 0 0, limit lower=0.0 upper=7.9 effort=1000.0 velocity=1.0
